File: Hardware/GISMo Board/SmartServo.kicad_pcb (KiCad board)
At the start: 2 copper layers, 18 x 22.4 mm, 46 parts, among them J2 I2C, M0 M+, M1 M-, U1 DRV8876RGTR, U2 STM32F302K8Ux

Commit message: Added head sink for motor driver
Parts:
- added HS1: HeatSink, TestPoint:TestPoint_Pad_2.0x2.0mm, B.Cu at (149.4, 104.9)
Connections:
- U1 pad 17: (no net) -> /DRV/HeatPad
